File: kicad-c128d/c128-u3-gal.kicad_pcb (KiCad board)
At the start: 2 copper layers, 21.5 x 37.3 mm, 5 parts, among them J1 Conn_02x04_Row_Letter_Last, J2 Conn_01x02, J3 Conn_01x04, U1 74LS138, U2 GAL20V10

Commit message: correct GAL device name to GAL22V10
Parts:
- U2: value GAL20V10 -> GAL22V10
Changed lines of the file:
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@@
       (effects (font (size 1 1) (thickness 0.15)))
     )
-    (fp_text value "GAL20V10" (at 3.825 13.975 90) (layer "F.SilkS")
+    (fp_text value "GAL22V10" (at 3.825 13.975 90) (layer "F.SilkS")
       (effects (font (size 1 1) (thickness 0.15)))
     )
